Commit message: Changed the home (zero) position of joint 2 to point up

File: src/ur_er9_support/er9.xacro (robot description, xacro)
@@ -25,9 +25,9 @@
         <link name="${link_name}"/>
     </xacro:macro>
-    <xacro:macro name="def_joint" params="joint_name type axis effort lower upper velocity origin parent child">
+    <xacro:macro name="def_joint" params="joint_name type axis effort lower upper velocity origin angle parent child">
         <joint name="${joint_name}" type="${type}">
             <axis xyz="${axis}"/>
             <limit effort="${effort}" lower="${lower*DEG2RAD}" upper="${upper*DEG2RAD}" velocity="${velocity}"/>
-            <origin rpy="0 0 0" xyz="${origin}"/>
+            <origin rpy="${angle}" xyz="${origin}"/>
             <parent link="${parent}"/>
             <child link="${child}"/>
@@ -44,17 +44,21 @@
     <xacro:def_link link_name="base_link" mesh_name="base.stl"/>
     <xacro:def_link link_name="link1" mesh_name="link1.stl"/>
-    <xacro:def_joint joint_name="joint1" type="revolute" axis="0 0 1" effort="1000.0" lower="-250" upper="250" velocity="1.0" origin="0 0 0.174"
+    <xacro:def_joint joint_name="joint1" type="revolute" axis="0 0 1" effort="1000.0" lower="-250" upper="250" velocity="1.0" origin="0 0 0.174" angle="0 0 0"
                      parent="base_link" child="link1"/>
     <xacro:def_link link_name="link2" mesh_name="link2.stl"/>
-    <xacro:def_joint joint_name="joint2" type="revolute" axis="0 1 0" effort="1000.0" lower="-150" upper="60" velocity="1.0" origin="0.07 -0.1 0.164"
+<!-- OLD JOINT 2 HOME (ZERO) CONFIGURATION -->
+<!--    <xacro:def_joint joint_name="joint2" type="revolute" axis="0 1 0" effort="1000.0" lower="-150" upper="60" velocity="1.0" origin="0.07 -0.1 0.164" angle="0 0 0"
+                     parent="link1" child="link2"/> -->
+<!-- New joint 2 home (zeroing) configuration-->
+    <xacro:def_joint joint_name="joint2" type="revolute" axis="0 1 0" effort="1000.0" lower="-60" upper="150" velocity="1.0" origin="0.07 -0.1 0.164" angle="0 ${-90*DEG2RAD} 0"
                      parent="link1" child="link2"/>
     <xacro:def_link link_name="link3" mesh_name="link3.stl"/>
-    <xacro:def_joint joint_name="joint3" type="revolute" axis="0 1 0" effort="1000.0" lower="-225" upper="225" velocity="1.0" origin="0.290 0.018 0"
+    <xacro:def_joint joint_name="joint3" type="revolute" axis="0 1 0" effort="1000.0" lower="-225" upper="225" velocity="1.0" origin="0.290 0.018 0" angle="0 0 0"
                      parent="link2" child="link3"/>
     <xacro:def_link link_name="link4" mesh_name="link4.stl"/>
-    <xacro:def_joint joint_name="joint4" type="revolute" axis="0 1 0" effort="1000.0" lower="-180" upper="180" velocity="1.0" origin="0.239 0.041 0"
+    <xacro:def_joint joint_name="joint4" type="revolute" axis="0 1 0" effort="1000.0" lower="-180" upper="180" velocity="1.0" origin="0.239 0.041 0" angle="0 0 0"
                      parent="link3" child="link4"/>
     <xacro:def_link link_name="link5" mesh_name="link5.stl"/>
-    <xacro:def_joint joint_name="joint5" type="revolute" axis="1 0 0" effort="1000.0" lower="-360" upper="360" velocity="1.0" origin="0.111 0 0"
+    <xacro:def_joint joint_name="joint5" type="revolute" axis="1 0 0" effort="1000.0" lower="-360" upper="360" velocity="1.0" origin="0.111 0 0" angle="0 0 0"
                      parent="link4" child="link5"/>
     <xacro:def_empty_link link_name="tool0"/>
@@ -65,7 +69,7 @@
     <xacro:def_fixed_joint joint_name="gripper_base_joint" origin="0 0 0" parent="tool0" child="gripper_base_link"/>
     <xacro:def_link link_name="gripper_base_link" mesh_name="ER9_Gripper_base.dae" />
-    <xacro:def_joint joint_name="gripper_left_joint" type="prismatic" axis="0 -1 0" effort="1000.0" lower="0" upper="1.8" velocity="1.0" origin="0 0 0" parent="gripper_base_link" child="gripper_left_link" />
+    <xacro:def_joint joint_name="gripper_left_joint" type="prismatic" axis="0 -1 0" effort="1000.0" lower="0" upper="1.8" velocity="1.0" origin="0 0 0" angle="0 0 0" parent="gripper_base_link" child="gripper_left_link" />
     <xacro:def_link link_name="gripper_left_link" mesh_name="ER9_Gripper_LC.dae" />
-    <xacro:def_joint joint_name="gripper_right_joint" type="prismatic" axis="0 1 0" effort="1000.0" lower="0" upper="1.8" velocity="1.0" origin="0 0 0" parent="gripper_base_link" child="gripper_right_link" />
+    <xacro:def_joint joint_name="gripper_right_joint" type="prismatic" axis="0 1 0" effort="1000.0" lower="0" upper="1.8" velocity="1.0" origin="0 0 0" angle="0 0 0" parent="gripper_base_link" child="gripper_right_link" />
     <xacro:def_link link_name="gripper_right_link" mesh_name="ER9_Gripper_RC.dae" />
 </robot>
